File: tool_switch.sch (KiCad schematic (older format))
At the start: 19 parts

Commit message: version with a relay
Parts:
- removed Q? (x3): Q_NMOS_DGS, symbol Q_NMOS_DGS
- removed R? (x5): R, symbol R
- added C1: 100nF, symbol C
- added R1, R2: 10k, symbol R
- D1: renamed from D?; value D_Schottky -> 1N60
- Q1: renamed from Q?; value Q_NPN_EBC -> BD578
- R3: renamed from R?; value R -> 330R
- R4: renamed from R?; value R -> 6.8k
- gave numbers to parts that had none: 7
Connections:
- net +9V: no longer U1.4
- net GND: now also C1.2, R1.1, R2.1
- net opt1: now also R4.2, U1.3, R2.2; no longer SW1.3
- net opt2: now also U1.4, R1.2
- net at Q1.2 (B), R4.1: now also C1.1
- net at Q1.3 (C): now also D1.2 (A), RL1.A2
- net opt4: no longer names the net of SW1.4
Other:
- moved on the sheet: D1, P1, P2, P3, P4, Q1, R3, R4, RL1, SW1, U1

Commit message: added pcb layout
Parts:
- removed RL1: FINDER-36.11.4001, symbol FINDER-36.11.4001
- removed SW1: SW_Rotary12, symbol SW_Rotary12
- added RL1: G5Q-2, Relays_THT:Relay_SANYOU_SRD_Series_Form_C, symbol G5Q-2
- C1: footprint (none) -> Capacitors_ThroughHole:C_Disc_D3.0mm_W1.6mm_P2.50mm
- D1: footprint (none) -> Diodes_THT:D_A-405_P7.62mm_Horizontal
- P1, P2, P3, P4: footprint (none) -> borniers:bornier2_V
- Q1: footprint (none) -> TO_SOT_Packages_THT:TO-92_Inline_Narrow_Oval
- R1, R2, R3, R4: footprint (none) -> Resistors_ThroughHole:R_Axial_DIN0204_L3.6mm_D1.6mm_P5.08mm_Horizontal
- U1: footprint DIP-4 -> Housings_DIP:DIP-4_W7.62mm_LongPads
Connections:
- net +9V: now also RL1.5
- net Ai: now also RL1.3
- net Ao: now also RL1.1
- net at D1.2 (A), Q1.3 (C): now also RL1.2
Changed lines of the file:
@@
 F 0 "U1" H 1600 3450 50  0000 L CNN
 F 1 "PC817" H 1800 3450 50  0000 L CNN
-F 2 "DIP-4" H 1600 3050 50  0000 L CIN
+F 2 "Housings_DIP:DIP-4_W7.62mm_LongPads" H 1600 3050 50  0000 L CIN
 F 3 "" H 1800 3250 50  0000 L CNN
 	1    1800 3250
@@
 F 0 "P4" V 700 3250 40  0000 C CNN
 F 1 "CONN_2" V 800 3250 40  0000 C CNN
-F 2 "" H 750 3250 60  0001 C CNN
+F 2 "borniers:bornier2_V" H 750 3250 60  0001 C CNN
 F 3 "" H 750 3250 60  0001 C CNN
 	1    750  3250
@@
 F 0 "R3" V 1380 3350 50  0000 C CNN
 F 1 "330R" V 1300 3350 50  0000 C CNN
-F 2 "" V 1230 3350 50  0000 C CNN
+F 2 "Resistors_ThroughHole:R_Axial_DIN0204_L3.6mm_D1.6mm_P5.08mm_Horizontal" V 1230 3350 50  0001 C CNN
 F 3 "" H 1300 3350 50  0000 C CNN
 	1    1300 3350
@@
 F 0 "P3" V 700 1800 40  0000 C CNN
 F 1 "CONN_2" V 800 1800 40  0000 C CNN
-F 2 "" H 750 1800 60  0001 C CNN
+F 2 "borniers:bornier2_V" H 750 1800 60  0001 C CNN
 F 3 "" H 750 1800 60  0001 C CNN
 	1    750  1800
@@
 F 0 "R4" V 2730 3350 50  0000 C CNN
 F 1 "6.8k" V 2650 3350 50  0000 C CNN
-F 2 "" V 2580 3350 50  0000 C CNN
+F 2 "Resistors_ThroughHole:R_Axial_DIN0204_L3.6mm_D1.6mm_P5.08mm_Horizontal" V 2580 3350 50  0001 C CNN
 F 3 "" H 2650 3350 50  0000 C CNN
 	1    2650 3350
@@
 F 0 "P2" V 700 1350 40  0000 C CNN
 F 1 "CONN_2" V 800 1350 40  0000 C CNN
-F 2 "" H 750 1350 60  0001 C CNN
+F 2 "borniers:bornier2_V" H 750 1350 60  0001 C CNN
 F 3 "" H 750 1350 60  0001 C CNN
 	1    750  1350
@@
 	2200 3150 2100 3150
 Wire Wire Line
-	2200 1750 2200 2400
-Wire Wire Line
-	2200 2400 2200 3150
+	2200 1750 2200 3150
 Wire Wire Line
 	3350 3900 3350 3550
 Wire Wire Line
-	2100 3350 2400 3350
-Wire Wire Line
-	2400 3350 2500 3350
+	2100 3350 2500 3350
 $Comp
 L Q_NPN_EBC Q1
@@
 F 0 "Q1" H 3450 3400 50  0000 L CNN
 F 1 "BD578" H 3450 3300 50  0000 L CNN
-F 2 "" H 3450 3450 50  0000 C CNN
+F 2 "TO_SOT_Packages_THT:TO-92_Inline_Narrow_Oval" H 3450 3450 50  0001 C CNN
 F 3 "" H 3250 3350 50  0000 C CNN
 	1    3250 3350
@@
 $EndComp
 $Comp
-L +9V #PWR02
+L +9V #PWR01
 U 1 1 5880E8AF
 P 3350 1650
-F 0 "#PWR02" H 3350 1500 50  0001 C CNN
+F 0 "#PWR01" H 3350 1500 50  0001 C CNN
 F 1 "+9V" H 3350 1790 50  0000 C CNN
 F 2 "" H 3350 1650 50  0000 C CNN
@@
 $EndComp
 Wire Wire Line
-	3100 1750 3350 1750
-Wire Wire Line
-	3350 1750 3650 1750
+	3100 1750 3650 1750
 Wire Wire Line
 	3100 1750 3100 1950
@@
 	3100 2250 3100 2450
 Wire Wire Line
-	3100 2450 3350 2450
-Wire Wire Line
-	3350 2450 3650 2450
+	3100 2450 3650 2450
 Wire Wire Line
 	3350 2450 3350 3150
 $Comp
-L +9V #PWR03
+L +9V #PWR02
 U 1 1 5881A2A9
 P 1250 1700
-F 0 "#PWR03" H 1250 1550 50  0001 C CNN
+F 0 "#PWR02" H 1250 1550 50  0001 C CNN
 F 1 "+9V" H 1250 1840 50  0000 C CNN
 F 2 "" H 1250 1700 50  0000 C CNN
@@
 $EndComp
 $Comp
-L GND #PWR04
+L GND #PWR03
 U 1 1 5881A2EE
 P 1250 1900
-F 0 "#PWR04" H 1250 1650 50  0001 C CNN
+F 0 "#PWR03" H 1250 1650 50  0001 C CNN
 F 1 "GND" H 1250 1750 50  0000 C CNN
 F 2 "" H 1250 1900 50  0000 C CNN
@@
 Wire Wire Line
 	1100 1450 1300 1450
-$Comp
-L FINDER-36.11.4001 RL1
-U 1 1 58822F34
-P 3850 2100
-F 0 "RL1" H 4300 2250 50  0000 L CNN
-F 1 "FINDER-36.11.4001" H 4300 2150 50  0000 L CNN
-F 2 "" H 3850 2100 50  0001 C CNN
-F 3 "" H 3850 2100 50  0001 C CNN
-	1    3850 2100
-	1    0    0    -1
-$EndComp
 Wire Wire Line
 	3650 1750 3650 1800
@@
 F 0 "D1" H 3100 2200 50  0000 C CNN
 F 1 "1N60" H 3100 2000 50  0000 C CNN
-F 2 "" H 3100 2100 50  0001 C CNN
+F 2 "Diodes_THT:D_A-405_P7.62mm_Horizontal" H 3100 2100 50  0001 C CNN
 F 3 "" H 3100 2100 50  0001 C CNN
 	1    3100 2100
@@
 F 0 "P1" V 700 950 40  0000 C CNN
 F 1 "CONN_2" V 800 950 40  0000 C CNN
-F 2 "" H 750 950 60  0001 C CNN
+F 2 "borniers:bornier2_V" H 750 950 60  0001 C CNN
 F 3 "" H 750 950 60  0001 C CNN
 	1    750  950
@@
 Wire Wire Line
 	1100 1050 1300 1050
-Text GLabel 3950 1650 1    60   Input ~ 0
+Text GLabel 4150 1650 1    60   Input ~ 0
 Ai
 Text GLabel 4050 2450 3    60   Input ~ 0
@@
 	4050 2400 4050 2450
 Wire Wire Line
-	3950 1650 3950 1800
+	4150 1650 4150 1800
 Text GLabel 4450 1650 1    60   Input ~ 0
 Bi
@@
 Wire Wire Line
 	4450 1650 4450 2450
-$Comp
-L SW_Rotary12 SW1
-U 1 1 5882377C
-P 5600 3950
-F 0 "SW1" H 5600 4650 50  0000 C CNN
-F 1 "SW_Rotary12" H 5600 3250 50  0000 C CNN
-F 2 "" H 5400 4650 50  0001 C CNN
-F 3 "" H 5400 4650 50  0001 C CNN
-	1    5600 3950
-	1    0    0    -1
-$EndComp
-Text GLabel 6100 3350 2    60   Input ~ 0
-opt1
-Text GLabel 6100 3450 2    60   Input ~ 0
-opt2
 Text GLabel 2400 1750 1    60   Input ~ 0
 opt1
-$Comp
-L +9V #PWR05
-U 1 1 5882430B
-P 5000 3950
-F 0 "#PWR05" H 5000 3800 50  0001 C CNN
-F 1 "+9V" H 5000 4090 50  0000 C CNN
-F 2 "" H 5000 3950 50  0000 C CNN
-F 3 "" H 5000 3950 50  0000 C CNN
-	1    5000 3950
-	0    -1   -1   0
-$EndComp
-Wire Wire Line
-	6000 3350 6100 3350
-Wire Wire Line
-	6000 3450 6100 3450
-Wire Wire Line
-	2400 1750 2400 2600
-Wire Wire Line
-	2400 2600 2400 3350
+Wire Wire Line
+	2400 1750 2400 3350
 Connection ~ 2400 3350
 Wire Wire Line
-	2800 3350 2950 3350
-Wire Wire Line
-	2950 3350 3050 3350
+	2800 3350 3050 3350
 Text GLabel 2200 1750 1    60   Input ~ 0
 opt2
@@
 F 0 "R2" V 2030 2600 50  0000 C CNN
 F 1 "10k" V 1950 2600 50  0000 C CNN
-F 2 "" V 1880 2600 50  0000 C CNN
+F 2 "Resistors_ThroughHole:R_Axial_DIN0204_L3.6mm_D1.6mm_P5.08mm_Horizontal" V 1880 2600 50  0001 C CNN
 F 3 "" H 1950 2600 50  0000 C CNN
 	1    1950 2600
@@
 F 0 "R1" V 2030 2400 50  0000 C CNN
 F 1 "10k" V 1950 2400 50  0000 C CNN
-F 2 "" V 1880 2400 50  0000 C CNN
+F 2 "Resistors_ThroughHole:R_Axial_DIN0204_L3.6mm_D1.6mm_P5.08mm_Horizontal" V 1880 2400 50  0001 C CNN
 F 3 "" H 1950 2400 50  0000 C CNN
 	1    1950 2400
@@
 Connection ~ 2400 2600
 $Comp
-L GND #PWR06
+L GND #PWR04
 U 1 1 5885BC17
 P 1600 2600
-F 0 "#PWR06" H 1600 2350 50  0001 C CNN
+F 0 "#PWR04" H 1600 2350 50  0001 C CNN
 F 1 "GND" H 1600 2450 50  0000 C CNN
 F 2 "" H 1600 2600 50  0000 C CNN
@@
 	1700 2400 1800 2400
 Wire Wire Line
-	1600 2600 1700 2600
-Wire Wire Line
-	1700 2600 1800 2600
+	1600 2600 1800 2600
 Connection ~ 1700 2600
 $Comp
@@
 F 0 "C1" H 2975 3750 50  0000 L CNN
 F 1 "100nF" H 2975 3550 50  0000 L CNN
-F 2 "" H 2988 3500 50  0001 C CNN
+F 2 "Capacitors_ThroughHole:C_Disc_D3.0mm_W1.6mm_P2.50mm" H 2988 3500 50  0001 C CNN
 F 3 "" H 2950 3650 50  0001 C CNN
 	1    2950 3650
@@
 Connection ~ 2950 3350
 $Comp
-L GND #PWR07
+L GND #PWR05
 U 1 1 58863E11
 P 2950 3950
-F 0 "#PWR07" H 2950 3700 50  0001 C CNN
+F 0 "#PWR05" H 2950 3700 50  0001 C CNN
 F 1 "GND" H 2950 3800 50  0000 C CNN
 F 2 "" H 2950 3950 50  0000 C CNN
@@
 $EndComp
 Wire Wire Line
-	2950 3800 2950 3900
-Wire Wire Line
-	2950 3900 2950 3950
+	2950 3800 2950 3950
 Wire Wire Line
 	2950 3900 3350 3900
 Connection ~ 2950 3900
+$Comp
+L G5Q-2 RL1
+U 1 1 588784A8
+P 3650 2300
+F 0 "RL1" H 4300 2650 50  0000 L CNN
+F 1 "G5Q-2" H 4300 2550 50  0000 L CNN
+F 2 "Relays_THT:Relay_SANYOU_SRD_Series_Form_C" H 4300 2450 50  0001 L CNN
+F 3 "" H 3850 2100 50  0001 C CNN
+	1    3650 2300
+	1    0    0    -1
+$EndComp
 $EndSCHEMATC
